File: Test Boards/AetherMesh Test Fixture Mezz/AetherMesh Test Fixture Mezz V1.0.brd (EAGLE design)
At the start: 71.2 x 57.5 mm, 7 parts, among them J1 POWER_JACKEJ508A, M1 AETHERMESH_MODULEMEZZ-HOLES

Commit message: Updated test boards with silkscreen pin names and current measurment jumper
Parts:
- added JP3: (no value), 1. growflux:1X02_LOCK
Connections:
- new net N$3: JP2.10, JP3.1, M1.P$17, M1.P$18
- net VCC: now also JP3.2; no longer JP2.10, M1.P$17, M1.P$18
Routing:
- net N$3: track 0.00 -> 51.0 mm
- net VCC: track 77.5 -> 39.8 mm, vias 2 -> 0
Other:
- board text added: "3V3 input"
- board text added: "CURRENT MEASUREMENT"
- board text added: "DIO0"
- board text added: "DIO1"
- board text added: "DIO10"
- board text added: "DIO11"
- board text added: "DIO12"
- board text added: "DIO13"
- board text added: "DIO14"
- board text added: "DIO2"
- board text added: "DIO3"
- board text added: "DIO4"
- board text added: "DIO7"
- board text added: "DIO8"
- board text added: "DIO9"
- board text added: "GND"
- board text added: "RST"
- board text added: "TCK"
- board text added: "TDI"
- board text added: "TDO"
- board text added: "TMS"
- board text added: "VCC"
Changed lines of the file:
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@@
 <?xml version="1.0" encoding="utf-8"?>
 <!DOCTYPE eagle SYSTEM "eagle.dtd">
-<eagle version="8.3.2">
+<eagle version="8.4.1">
 <drawing>
 <settings>
@@
 <rectangle x1="30.87878125" y1="12.143740625" x2="40.62221875" y2="12.179296875" layer="21"/>
 <rectangle x1="30.87878125" y1="12.1793" x2="40.62221875" y2="12.21485625" layer="21"/>
+<text x="59.2836" y="26.9748" size="1.27" layer="21" font="vector">3V3 input</text>
+<text x="50.3936" y="16.3068" size="1.27" layer="21" font="vector" align="center">CURRENT
+MEASUREMENT</text>
+<text x="1.6256" y="50.8508" size="0.8128" layer="21" font="vector" ratio="12" align="center">TMS</text>
+<text x="1.6256" y="48.3108" size="0.8128" layer="21" font="vector" ratio="12" align="center">TCK</text>
+<text x="1.6256" y="45.7708" size="0.8128" layer="21" font="vector" ratio="12" align="center">TDO</text>
+<text x="1.6256" y="43.2308" size="0.8128" layer="21" font="vector" ratio="12" align="center">TDI</text>
+<text x="1.6256" y="40.6908" size="0.8128" layer="21" font="vector" ratio="12" align="center">RST</text>
+<text x="1.6256" y="38.1508" size="0.8128" layer="21" font="vector" ratio="12" align="center">DIO7</text>
+<text x="1.6256" y="35.6108" size="0.8128" layer="21" font="vector" ratio="12" align="center">DIO8</text>
+<text x="1.6256" y="33.0708" size="0.8128" layer="21" font="vector" ratio="12" align="center">DIO9</text>
+<text x="1.6256" y="30.5308" size="0.8128" layer="21" font="vector" ratio="12" align="center">DIO10</text>
+<text x="1.6256" y="27.4828" size="0.8128" layer="21" font="vector" ratio="12" align="center">GND
+</text>
+<text x="47.5996" y="53.8988" size="0.8128" layer="21" font="vector" ratio="12" align="top-left">DIO14</text>
+<text x="47.5996" y="51.6128" size="0.8128" layer="21" font="vector" ratio="12" align="top-left">DIO13</text>
+<text x="47.5996" y="49.0728" size="0.8128" layer="21" font="vector" ratio="12" align="top-left">DIO12</text>
+<text x="47.5996" y="46.2788" size="0.8128" layer="21" font="vector" ratio="12" align="top-left">DIO11</text>
+<text x="47.5996" y="43.7388" size="0.8128" layer="21" font="vector" ratio="12" align="top-left">DIO4</text>
+<text x="47.5996" y="41.1988" size="0.8128" layer="21" font="vector" ratio="12" align="top-left">DIO3</text>
+<text x="47.5996" y="38.6588" size="0.8128" layer="21" font="vector" ratio="12" align="top-left">DIO0</text>
+<text x="47.5996" y="36.1188" size="0.8128" layer="21" font="vector" ratio="12" align="top-left">DIO1</text>
+<text x="47.5996" y="33.5788" size="0.8128" layer="21" font="vector" ratio="12" align="top-left">DIO2</text>
+<text x="47.5996" y="31.0388" size="0.8128" layer="21" font="vector" ratio="12" align="top-left">VCC</text>
 </plain>
 <attributes>
@@
 <param name="dpMaxLengthDifference" value="10mm"/>
 <param name="dpGapFactor" value="2.5"/>
-<param name="checkGrid" value="0"/>
 <param name="checkAngle" value="0"/>
 <param name="checkFont" value="1"/>
 <param name="checkRestrict" value="1"/>
+<param name="checkStop" value="0"/>
 <param name="useDiameter" value="13"/>
 <param name="maxErrors" value="50"/>
@@
 <attribute name="MFG#" value="9774040243R" x="13.1445" y="28.6766" size="1.778" layer="27" display="off"/>
 </element>
+<element name="JP3" library="1. growflux" package="1X02_LOCK" value="" x="49.8856" y="22.352" smashed="yes" rot="R270">
+<attribute name="VALUE" x="46.7106" y="23.622" size="1.27" layer="27" rot="R270"/>
+</element>
 </elements>
 <signals>
@@
 <wire x1="20.6756" y1="18.2372" x2="20.701" y2="18.2626" width="0.1524" layer="1"/>
 <wire x1="20.701" y1="18.2626" x2="21.844" y2="19.2024" width="0.1524" layer="1"/>
-<contactref element="JP2" pad="10"/>
 <wire x1="21.844" y1="19.2024" x2="22.606" y2="19.812" width="0.4064" layer="1"/>
-<wire x1="45.466" y1="30.5308" x2="45.4152" y2="30.5816" width="0.8128" layer="1"/>
-<contactref element="M1" pad="P$17"/>
-<contactref element="M1" pad="P$18"/>
-<wire x1="45.4406" y1="30.5562" x2="45.4406" y2="30.5816" width="0.8128" layer="1"/>
-<wire x1="45.4406" y1="30.5562" x2="41.6052" y2="26.7208" width="0.8128" layer="1"/>
-<wire x1="23.384446875" y1="26.7208" x2="41.6052" y2="26.7208" width="0.8128" layer="1"/>
-<wire x1="11.462" y1="37.005" x2="10.2842" y2="37.005" width="0.254" layer="1"/>
-<wire x1="10.051575" y1="36.734540625" x2="10.2842" y2="37.005" width="0.254" layer="1"/>
-<wire x1="10.051575" y1="36.734540625" x2="9.3472" y2="35.9156" width="0.254" layer="1"/>
-<wire x1="9.3472" y1="35.9156" x2="9.3472" y2="35.7632" width="0.254" layer="1"/>
-<wire x1="10.2866875" y1="37.505" x2="11.462" y2="37.505" width="0.254" layer="1"/>
-<wire x1="10.2866875" y1="37.505" x2="10.2866875" y2="36.969653125" width="0.254" layer="1"/>
-<wire x1="10.2866875" y1="36.969653125" x2="10.051575" y2="36.734540625" width="0.254" layer="1"/>
-<wire x1="58.7724" y1="19.812" x2="56.2102" y2="19.812" width="0.8128" layer="16"/>
-<wire x1="56.2102" y1="19.812" x2="45.4406" y2="30.5816" width="0.8128" layer="16"/>
-<wire x1="22.606" y1="19.812" x2="22.606" y2="20.828" width="0.8128" layer="1"/>
-<via x="22.606" y="20.828" extent="1-16" drill="0.7"/>
-<wire x1="22.606" y1="20.828" x2="22.606" y2="28.5496" width="0.8128" layer="16"/>
-<via x="22.606" y="28.5496" extent="1-16" drill="0.7"/>
-<wire x1="22.606" y1="28.5496" x2="22.606" y2="27.466353125" width="0.8128" layer="1"/>
-<wire x1="22.606" y1="27.466353125" x2="23.384446875" y2="26.7208" width="0.8128" layer="1"/>
-<wire x1="9.3472" y1="35.7632" x2="9.3472" y2="33.5153" width="0.8128" layer="1"/>
-<wire x1="9.3472" y1="33.5153" x2="10.4902" y2="32.3723" width="0.8128" layer="1"/>
-<wire x1="10.4902" y1="32.3723" x2="18.7833" y2="32.3723" width="0.8128" layer="1"/>
-<wire x1="18.7833" y1="32.3723" x2="22.606" y2="28.5496" width="0.8128" layer="1"/>
-<wire x1="45.4406" y1="30.5816" x2="45.4152" y2="30.5816" width="0" layer="19" extent="1-16"/>
+<wire x1="23.8252" y1="20.828" x2="22.606" y2="19.812" width="0.8128" layer="1"/>
+<contactref element="JP3" pad="2"/>
+<wire x1="58.7724" y1="19.812" x2="50.0634" y2="19.812" width="0.8128" layer="1"/>
+<wire x1="50.0634" y1="19.812" x2="49.8856" y2="19.6342" width="0.8128" layer="1"/>
+<wire x1="49.8856" y1="19.6342" x2="48.6918" y2="20.828" width="0.8128" layer="1"/>
+<wire x1="48.6918" y1="20.828" x2="23.8252" y2="20.828" width="0.8128" layer="1"/>
 </signal>
 <signal name="N$2">
@@
 <wire x1="16.4606" y1="41.5304" x2="17.6276" y2="42.545" width="0.1524" layer="1"/>
 </signal>
+<signal name="N$3">
+<contactref element="JP2" pad="10"/>
+<contactref element="M1" pad="P$17"/>
+<contactref element="M1" pad="P$18"/>
+<contactref element="JP3" pad="1"/>
+<wire x1="11.462" y1="37.505" x2="11.462" y2="37.005" width="0.254" layer="1"/>
+<wire x1="11.462" y1="37.005" x2="10.2842" y2="37.005" width="0.254" layer="1"/>
+<wire x1="10.2842" y1="37.005" x2="9.9568" y2="36.6776" width="0.254" layer="1"/>
+<wire x1="9.9568" y1="36.6776" x2="9.9568" y2="35.052" width="0.8128" layer="1"/>
+<wire x1="9.9568" y1="35.052" x2="10.5664" y2="34.4424" width="0.8128" layer="1"/>
+<wire x1="10.5664" y1="34.4424" x2="11.14231875" y2="34.4424" width="0.8128" layer="1"/>
+<wire x1="14.43775625" y1="34.3662" x2="14.46035625" y2="34.3436" width="0.8128" layer="1"/>
+<wire x1="20.9268" y1="34.3436" x2="24.6888" y2="30.5816" width="0.8128" layer="1"/>
+<wire x1="14.46035625" y1="34.3436" x2="20.9268" y2="34.3436" width="0.8128" layer="1"/>
+<wire x1="11.14231875" y1="34.4424" x2="11.21851875" y2="34.3662" width="0.8128" layer="1"/>
+<wire x1="11.21851875" y1="34.3662" x2="14.43775625" y2="34.3662" width="0.8128" layer="1"/>
+<wire x1="24.6888" y1="30.5816" x2="45.4406" y2="30.5816" width="0.8128" layer="1"/>
+<wire x1="45.4406" y1="30.5816" x2="49.8856" y2="26.1366" width="0.8128" layer="16"/>
+<wire x1="49.8856" y1="26.1366" x2="49.8856" y2="22.5298" width="0.8128" layer="16"/>
+</signal>
 </signals>
