File: Reference Designs/AA Sensor Board Reference Design.brd (EAGLE design)
At the start: 70.6 x 48.1 mm, 21 parts, among them IC1 TPS62730, M2 AETHERMESH_MODULEMEZZ-HOLES

Commit message: Updated AA sensor board reference design
Parts:
- removed C1, C3: 10uF, 2. growflux:C0805
- removed C2, C4: 2.2uF, 2. growflux:C0402
- removed IC1: TPS62730, 3. growflux:SON-6
- removed L1: 2.2uH, 2. growflux:0805
Connections:
- removed net L1: IC1.2, L1.1
- removed net STAT: IC1.1
- net DIO10: no longer IC1.5
- net GND: no longer C1.P$2, C2.P$1, C3.P$2, C4.P$1, IC1.4
- net N$4: now also JP1.P$1; no longer C4.P$2, IC1.6, L1.2
- net VBAT: no longer C1.P$1, C2.P$2, C3.P$1, IC1.3, JP1.P$1
Routing:
- net VBAT: track 9.00 -> 0.00 mm
- net DIO10: track 55.1 -> 52.6 mm, vias 2 -> 1
- net STAT: track 1.10 -> 0.00 mm, vias 1 -> 0
- removed copper zone on layer 1, net L1
- removed copper zone on layer 1, net N$4
- removed copper zone on layer 1, net VBAT
Changed lines of the file:
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@@
 <?xml version="1.0" encoding="utf-8"?>
 <!DOCTYPE eagle SYSTEM "eagle.dtd">
-<eagle version="8.4.1">
+<eagle version="8.6.0">
 <drawing>
 <settings>
@@
 <param name="checkRestrict" value="1"/>
 <param name="checkStop" value="0"/>
+<param name="checkValues" value="0"/>
 <param name="useDiameter" value="29"/>
 <param name="maxErrors" value="50"/>
@@
 <attribute name="MFG#" value="9774040243R" x="7.7403" y="-5.0284" size="1.778" layer="27" display="off"/>
 </element>
-<element name="C1" library="2. growflux" package="C0805" value="10uF" x="-7.7928" y="18.9684" smashed="yes" rot="R180">
-<attribute name="ALT#" value="GRM21BR71A106MA73L" x="-2.7128" y="18.9684" size="1.778" layer="27" rot="R180" display="off"/>
-<attribute name="MFG#" value="MF-CAP-1206-10UF" x="-2.7128" y="18.9684" size="1.778" layer="27" rot="R180" display="off"/>
-<attribute name="NAME" x="-5.5336" y="18.4428" size="0.8128" layer="25" font="vector" ratio="12"/>
-</element>
-<element name="IC1" library="3. growflux" package="SON-6" package3d_urn="urn:adsk.eagle:package:208239/1" value="TPS62730" x="-7.3864" y="13.4312" smashed="yes" rot="R90">
-<attribute name="MFG#" value="TPS62730DRYR" x="-16.2764" y="7.0812" size="1.778" layer="27" rot="R90" display="off"/>
-<attribute name="NAME" x="-7.6785" y="12.1485" size="0.8128" layer="21" font="vector" ratio="12" rot="R270"/>
-</element>
-<element name="L1" library="2. growflux" package="0805" value="2.2uH" x="-4.948" y="12.466" smashed="yes" rot="R270">
-<attribute name="ALT#" value="CKP2012N2R2M-T" x="0.132" y="18.816" size="1.778" layer="27" rot="R270" display="off"/>
-<attribute name="MFG#" value="LQM21PN2R2NGC" x="0.132" y="18.816" size="1.778" layer="27" rot="R270" display="off"/>
-<attribute name="NAME" x="-4.1225" y="13.6344" size="0.8128" layer="25" font="vector" ratio="12" rot="R270"/>
-</element>
-<element name="C2" library="2. growflux" package="C0402" value="2.2uF" x="-7.3864" y="15.3108" smashed="yes">
-<attribute name="ALT#" value="04026D225KAT2A" x="-12.4664" y="20.3908" size="1.778" layer="27" display="off"/>
-<attribute name="MFG#" value="CC0402KRX5R5BB225" x="-12.4664" y="20.3908" size="1.778" layer="27" display="off"/>
-<attribute name="NAME" x="-5.9464" y="14.8868" size="0.8128" layer="25" font="vector" ratio="12"/>
-</element>
-<element name="C3" library="2. growflux" package="C0805" value="10uF" x="-7.7928" y="16.9364" smashed="yes" rot="R180">
-<attribute name="ALT#" value="GRM21BR71A106MA73L" x="-2.7128" y="25.8264" size="1.778" layer="27" rot="R180" display="off"/>
-<attribute name="MFG#" value="MF-CAP-1206-10UF" x="-2.7128" y="25.8264" size="1.778" layer="27" rot="R180" display="off"/>
-<attribute name="NAME" x="-5.7368" y="16.614" size="0.8128" layer="25" font="vector" ratio="12"/>
-</element>
-<element name="C4" library="2. growflux" package="C0402" value="2.2uF" x="-9.266" y="13.3804" smashed="yes" rot="R270">
-<attribute name="ALT#" value="04026D225KAT2A" x="-18.156" y="22.2704" size="1.778" layer="27" rot="R270" display="off"/>
-<attribute name="MFG#" value="CC0402KRX5R5BB225" x="-18.156" y="22.2704" size="1.778" layer="27" rot="R270" display="off"/>
-<attribute name="NAME" x="-10.9756" y="11.2292" size="0.8128" layer="25" font="vector" ratio="12"/>
-</element>
 <element name="D2" library="MF_LEDs" package="PLCC4" value="" x="37.784" y="13.8518" rot="R270">
 <attribute name="MFG#" value="MF-LED-3228-RGB" x="37.784" y="13.8518" size="1.778" layer="27" rot="R270" display="off"/>
@@
 <contactref element="S3" pad="P$1"/>
 <contactref element="S4" pad="P$1"/>
-<contactref element="C3" pad="P$2"/>
-<contactref element="C1" pad="P$2"/>
-<contactref element="C2" pad="P$1"/>
-<contactref element="IC1" pad="4"/>
-<contactref element="C4" pad="P$1"/>
 <contactref element="JP2" pad="P$1"/>
 <contactref element="M2" pad="P$26"/>
@@
 <via x="24.9936" y="10.4648" extent="1-16" drill="0.3048"/>
 <via x="-4.4704" y="23.0632" extent="1-16" drill="0.3048"/>
-<wire x1="-16.0528" y1="7.8232" x2="-12.7614" y2="7.0396" width="0" layer="19" extent="1-1"/>
 <via x="17.78" y="-1.4224" extent="1-16" drill="0.3048"/>
 <via x="36.4744" y="-1.1176" extent="1-16" drill="0.3048"/>
@@
 <via x="10.16" y="1.3208" extent="1-16" drill="0.3048"/>
 <via x="15.24" y="10.4648" extent="1-16" drill="0.3048"/>
+<wire x1="-16.0528" y1="7.8232" x2="-12.7614" y2="7.0396" width="0" layer="19" extent="1-1"/>
 </signal>
 <signal name="N$3">
@@
 </signal>
 <signal name="VBAT">
-<contactref element="IC1" pad="3"/>
-<contactref element="C2" pad="P$2"/>
-<contactref element="C1" pad="P$1"/>
-<contactref element="C3" pad="P$1"/>
-<polygon width="0.1524" layer="1" isolate="0.1524" thermals="no">
-<vertex x="-6.472" y="15.9712"/>
-<vertex x="-6.472" y="13.9392"/>
-<vertex x="-6.5482" y="13.863"/>
-<vertex x="-7.0562" y="13.863"/>
-<vertex x="-7.0562" y="14.244"/>
-<vertex x="-7.2848" y="14.4472"/>
-<vertex x="-7.2848" y="15.9712"/>
-</polygon>
-<contactref element="JP1" pad="P$1"/>
-<wire x1="-6.8428" y1="18.9684" x2="-6.8428" y2="16.9364" width="0.6096" layer="1"/>
-<wire x1="-6.8428" y1="16.9364" x2="-6.8428" y2="15.3172" width="0.254" layer="1"/>
-<wire x1="-6.8428" y1="15.3172" x2="-6.8364" y2="15.3108" width="0.254" layer="1"/>
 <contactref element="TC2" pad="9"/>
-<wire x1="-2.794" y1="21.209" x2="-5.207" y2="21.209" width="0.6096" layer="1"/>
-<wire x1="-5.207" y1="21.209" x2="-6.858" y2="19.558" width="0.6096" layer="1"/>
-<wire x1="-6.858" y1="19.558" x2="-6.858" y2="18.9836" width="0.6096" layer="1"/>
-<wire x1="-6.858" y1="18.9836" x2="-6.8428" y2="18.9684" width="0.6096" layer="1"/>
-<wire x1="-6.8914" y1="13.9312" x2="-11.4914" y2="7.0396" width="0" layer="19" extent="1-1"/>
-</signal>
-<signal name="L1">
-<contactref element="IC1" pad="2"/>
-<contactref element="L1" pad="1"/>
-<polygon width="0.1524" layer="1" isolate="0.1524" thermals="no">
-<vertex x="-7.0816" y="13.5328"/>
-<vertex x="-6.3704" y="13.5328"/>
-<vertex x="-6.0656" y="13.8376"/>
-<vertex x="-4.3384" y="13.8376"/>
-<vertex x="-4.3384" y="12.9232"/>
-<vertex x="-6.0656" y="12.9232"/>
-<vertex x="-6.472" y="13.3296"/>
-<vertex x="-7.0816" y="13.3296"/>
-</polygon>
-</signal>
-<signal name="STAT">
-<contactref element="IC1" pad="1"/>
-<wire x1="-6.8914" y1="12.9312" x2="-6.403609375" y2="12.443409375" width="0.1524" layer="1"/>
-<wire x1="-6.403609375" y1="12.443409375" x2="-5.992209375" y2="12.443409375" width="0.1524" layer="1"/>
-<via x="-5.992209375" y="12.443409375" extent="1-16" drill="0.3048"/>
 </signal>
 <signal name="DIO2">
@@
 <signal name="DIO10">
 <contactref element="M2" pad="P$20"/>
-<contactref element="IC1" pad="5"/>
-<wire x1="-7.8814" y1="13.4312" x2="-10.3328" y2="13.4312" width="0.1524" layer="1"/>
-<via x="-10.3328" y="13.4312" extent="1-16" drill="0.3048"/>
 <contactref element="U$2" pad="15"/>
 <wire x1="47.6504" y1="11.11758125" x2="47.6504" y2="8.636" width="0.1524" layer="16"/>
@@
 <wire x1="15.37151875" y1="13.73601875" x2="34.259675" y2="13.73601875" width="0.1524" layer="16"/>
 <wire x1="45.01388125" y1="13.7541" x2="47.6504" y2="11.11758125" width="0.1524" layer="16"/>
-<wire x1="-7.8814" y1="13.4312" x2="6.0578" y2="4.8" width="0" layer="19" extent="1-1"/>
 </signal>
 <signal name="DIO9">
@@
 </signal>
 <signal name="N$4">
-<contactref element="IC1" pad="6"/>
-<contactref element="L1" pad="2"/>
-<contactref element="C4" pad="P$2"/>
 <contactref element="JP3" pad="1"/>
-<polygon width="0.1524" layer="1" isolate="0.1524" thermals="no">
-<vertex x="-4.3384" y="12.0088"/>
-<vertex x="-4.3384" y="11.196"/>
-<vertex x="-4.44" y="11.0944"/>
-<vertex x="-8.0976" y="11.0944"/>
-<vertex x="-9.6216" y="12.6184"/>
-<vertex x="-9.6216" y="13.1264"/>
-<vertex x="-9.012" y="13.1264"/>
-<vertex x="-9.012" y="13.0248"/>
-<vertex x="-8.0976" y="12.1104"/>
-<vertex x="-8.0976" y="13.0248"/>
-<vertex x="-7.6912" y="13.0248"/>
-<vertex x="-7.6912" y="12.5168"/>
-<vertex x="-7.1832" y="12.0088"/>
-</polygon>
 <wire x1="-0.982" y1="15.459" x2="-0.627" y2="15.104" width="0.6096" layer="1"/>
-<wire x1="-4.948" y1="11.566" x2="-3.42" y2="11.566" width="0.6096" layer="1"/>
-<wire x1="-2.794" y1="12.192" x2="-2.794" y2="13.462" width="0.6096" layer="1"/>
-<wire x1="-2.794" y1="13.462" x2="-0.982" y2="15.274" width="0.6096" layer="1"/>
 <wire x1="-0.982" y1="15.274" x2="-0.982" y2="15.459" width="0.6096" layer="1"/>
-<wire x1="-3.42" y1="11.566" x2="-2.794" y2="12.192" width="0.6096" layer="1"/>
+<contactref element="JP1" pad="P$1"/>
+<wire x1="-0.982" y1="15.459" x2="-0.982" y2="16.80756875" width="0.6096" layer="1"/>
+<wire x1="-2.794" y1="18.61956875" x2="-2.794" y2="21.209" width="0.6096" layer="1"/>
+<wire x1="-0.982" y1="16.80756875" x2="-2.794" y2="18.61956875" width="0.6096" layer="1"/>
 </signal>
 <signal name="N$1">
