File: Reference Designs/AA Sensor Board Reference Design.brd (EAGLE design)
At the start: 70.6 x 48.1 mm, 15 parts, among them M2 AETHERMESH_MODULEMEZZ-HOLES

Commit message: Final revisions to AA sensor reference design for production V1.0
Parts:
- removed TC2: TC2050-IDC, TagConnect:TC2050-IDC
- removed U$1: SENSOR_HUMIDITY_HDC2010, 3. growflux:HDC2010
- added IC1: SENSOR_HUMIDITY_HDC2010, 3. growflux:HDC2010
- added R1, R5: 10K, 3. growflux:R0402
- added TC1: DNP, TagConnect:TC2050-IDC
- added U$3: (no value), SparkFun-Aesthetics:OSHW-LOGO-L
- JP1, JP2: value M01BAT_SLOT -> DNP
- JP3: value (none) -> DNP
- M2: value AETHERMESH_MODULEMEZZ-HOLES -> AETHERMESH_MODULEMEZZ-NOHOLES; device AetherConnectivity:AETHERMESH_MEZZ_MOUNT_HOLES -> AetherConnectivity:AETHERMESH_MEZZ_MOUNT_NOHOLES
- U$2: value M10X22X10_LOCK -> DNP
- moved C5 21.5 mm to (40.1, 20.4)
- moved R8 4.42 mm to (7.94, -0.75)
- moved D2 0.81 mm to (38.6, 13.9)
- moved R4 0.81 mm to (41.1, 12.6)
- moved R2 0.81 mm to (38.5, 10.4)
- moved R3 0.81 mm to (36.0, 14.8)
Connections:
- removed net RX: TC2.5
- removed net TX: TC2.7
- removed net VBAT: TC2.9
- net DIO7: now also IC1.A2, R5.P$2; no longer U$1.A2
- net DIO8: now also IC1.B2, R1.P$2; no longer U$1.B2
- net GND: now also IC1.B1, IC1.C1, TC1.3, TC1.5, TC1.9; no longer TC2.10, TC2.3, U$1.C1
- net RESET: now also TC1.10; no longer TC2.2
- net TCK: now also TC1.4; no longer TC2.8
- net TDI: now also TC1.8; no longer TC2.4
- net TDO: now also TC1.6; no longer TC2.6
- net TMS: now also TC1.2; no longer TC2.1
- net VCC: now also IC1.A1, R1.P$1, R5.P$1, TC1.1; no longer U$1.A1
Routing:
- net VCC: track 73.4 -> 109.6 mm
- net TCK: track 49.0 -> 81.1 mm, vias 0 -> 2
- net DIO7: track 43.3 -> 72.9 mm, vias 0 -> 1
- net RESET: track 43.9 -> 73.1 mm, vias 0 -> 2
- net DIO8: track 43.1 -> 70.8 mm, vias 0 -> 1
- net TMS: track 51.0 -> 77.0 mm, vias 0 -> 2
- net TDO: track 47.2 -> 72.9 mm, vias 0 -> 2
- net TDI: track 45.0 -> 69.7 mm, vias 0 -> 2
- net GND: track 15.2 -> 20.6 mm, vias 38 -> 42
- net G2: track 0.00 -> 1.92 mm
- net B2: track 0.00 -> 1.90 mm
- net R2: track 0.00 -> 1.81 mm
- net N$4: track 7.19 -> 6.69 mm
Other:
- outline, holes or cut-outs redrawn
- board text added: "HDC2010 Humidity Sensor"
- board text added: "cut to measure current"

Commit message: Updated reference designs and test boards with latest XDS programmer tag connect header
Parts:
- removed TC1: DNP, TagConnect:TC2050-IDC
- added TC3: TC2050-IDC, TagConnect:TC2050-IDC
Connections:
- net DIO0: now also TC3.5
- net DIO1: now also TC3.7
- net GND: now also TC3.3, TC3.9; no longer TC1.3, TC1.5, TC1.9
- net RESET: now also TC3.10; no longer TC1.10
- net TCK: now also TC3.4; no longer TC1.4
- net TDI: now also TC3.8; no longer TC1.8
- net TDO: now also TC3.6; no longer TC1.6
- net TMS: now also TC3.2; no longer TC1.2
- net VCC: now also TC3.1; no longer TC1.1
Routing:
- net DIO0: track 47.3 -> 70.9 mm, vias 1 -> 3
- net DIO1: track 48.1 -> 67.8 mm, vias 1 -> 3
- net TCK: track 81.1 -> 83.6 mm
- net TDO: track 72.9 -> 74.9 mm
- net TMS: track 77.0 -> 78.5 mm
- net GND: track 20.6 -> 21.7 mm, vias 42 -> 43
- net RESET: track 73.1 -> 72.5 mm
